File: eternal-keypad.kicad_pcb (KiCad board)
At the start: 2 copper layers, 169.9 x 95.3 mm, 77 parts

Commit message: First prototype ready
Parts:
- removed Blade (x2): LOGO, Symbol:excalibur-blade
- removed Handle (x2): LOGO, Symbol:excalibur-handle
- added ?: , , F.Cu at (89.7, 31.8)
- added G***: LOGO, Symbol:eternal-logo-8mm, B.Cu at (53.0, 49.1)
- added G***: LOGO, Symbol:eternal-logo-8mm, F.Cu at (53.1, 49.1)
- added REF**: MountingHole_2.2mm_M2, MountingHole:MountingHole_2.2mm_M2, F.Cu at (103.2, 58.7)
- added REF**: MountingHole_2.2mm_M2, MountingHole:MountingHole_2.2mm_M2, F.Cu at (79.4, 115.9)
- added REF**: MountingHole_2.2mm_M2, MountingHole:MountingHole_2.2mm_M2, F.Cu at (198.4, 115.9)
- added REF**: MountingHole_2.2mm_M2, MountingHole:MountingHole_2.2mm_M2, F.Cu at (198.4, 58.7)
- D1, D10, D11, D12, D13, D14, D15, D16, D17, D18, D19, D2, D20, D21, D22, D23, D24, D25, D26, D27, D28, D29, D3, D30, D31, D32, D33, D34, D35, D36, D4, D5, D6, D7, D8, D9: footprint Diode_THT:D_DO-35_SOD27_P7.62mm_Horizontal -> Diode_THT:D_DO-35_SOD27_P7.62mm_Horizontal_Reversible
Other:
- board text added: "ETERNAL Keypad — Designed by Kyek in Italy"
- board text added: "V0.1α"
- board text removed: "ETERNAL Keypad V0.1α - Designed by Kyek in Italy"

Commit message: Update PCB and add firmware
Parts:
- removed the REF** at (103.2, 58.7)
- removed the REF** at (79.4, 115.9)
- removed the REF** at (198.4, 115.9)
- added REF**: MountingHole_2.2mm_M2_Pad_Via, MountingHole:MountingHole_2.2mm_M2_Pad_Via, F.Cu at (198.4, 115.9)
- added REF**: MountingHole_2.2mm_M2_Pad_Via, MountingHole:MountingHole_2.2mm_M2_Pad_Via, F.Cu at (103.2, 58.7)
- added REF**: MountingHole_2.2mm_M2_Pad_Via, MountingHole:MountingHole_2.2mm_M2_Pad_Via, F.Cu at (79.4, 115.9)
- REF**: value MountingHole_2.2mm_M2 -> MountingHole_2.2mm_M2_Pad_Via; footprint MountingHole:MountingHole_2.2mm_M2 -> MountingHole:MountingHole_2.2mm_M2_Pad_Via
Other:
- board text added: "ETERNAL Keypad Designed by Kyek in Italy"
- board text added: "R0"
- board text added: "V0.2α"
- board text removed: "ETERNAL Keypad — Designed by Kyek in Italy"
- board text removed: "V0.1α"

Commit message: Add plates and bump version
Parts:
- removed the REF** at (198.4, 115.9)
- removed the REF** at (103.2, 58.7)
- removed the REF** at (79.4, 115.9)
- removed the REF** at (198.4, 58.7)
- added REF**: MountingHole_3.2mm_M3_Pad_Via, MountingHole:MountingHole_3.2mm_M3_Pad_Via, F.Cu at (79.4, 115.9)
- added REF**: MountingHole_3.2mm_M3_Pad_Via, MountingHole:MountingHole_3.2mm_M3_Pad_Via, F.Cu at (102.4, 58.7)
- added REF**: MountingHole_3.2mm_M3_Pad_Via, MountingHole:MountingHole_3.2mm_M3_Pad_Via, F.Cu at (198.4, 115.9)
- added REF**: MountingHole_3.2mm_M3_Pad_Via, MountingHole:MountingHole_3.2mm_M3_Pad_Via, F.Cu at (198.4, 58.7)
- MX33: footprint MX_Only:MXOnly-1U-Reversible-NoLED -> MX_Only:MXOnly-1.25U-Reversible-NoLED
- MX35: footprint MX_Only:MXOnly-3U-Reversible-ReversedStabilizers-NoLED -> MX_Only:MXOnly-2.75U-Reversible-ReversedStabilizers-NoLED
- moved MX34 4.76 mm to (136.5, 125.4)
- moved MX33 2.38 mm to (115.1, 125.4)
- moved MX35 2.38 mm to (172.2, 125.4)
- moved D15 0.79 mm to (73.8, 91.3)
- moved D23 0.79 mm to (73.8, 110.3)
- moved D31 0.79 mm to (73.8, 129.4)
Routing:
- net GND: track 18.8 -> 0.00 mm
- net COL1: track 139.9 -> 128.0 mm
- net Net-(D34-Pad2): track 12.7 -> 17.4 mm
- net COL7: track 255.8 -> 252.3 mm
- net COL5: track 216.1 -> 218.6 mm
- net Net-(D33-Pad2): track 12.7 -> 15.0 mm
- net Net-(D35-Pad2): track 12.7 -> 15.0 mm
- net COL3: track 182.5 -> 184.3 mm
- net COL6: track 206.9 -> 208.2 mm
- net COL2: track 164.1 -> 165.0 mm
- net Net-(D15-Pad2): track 12.7 -> 13.5 mm
- net Net-(D31-Pad2): track 12.7 -> 13.5 mm
- net Net-(D23-Pad2): track 12.7 -> 13.5 mm
- net ROW2: track 168.3 -> 167.6 mm
- net ROW0: track 146.2 -> 145.6 mm
Other:
- board text added: "V1.0"
- board text removed: "V0.2α"

Commit message: Final adjustments and case patterns
Parts:
- removed the REF** at (79.4, 115.9)
- removed the REF** at (102.4, 58.7)
- added REF**: MountingHole_4.6mm_Pad_Via, MountingHole:MountingHole_4.6mm_Pad_Via_Custom, F.Cu at (79.4, 115.9)
- added REF**: MountingHole_4.6mm_Pad_Via, MountingHole:MountingHole_4.6mm_Pad_Via_Custom, F.Cu at (102.4, 58.7)
- FACE DOWN: value ProMicro -> ProMicro-Reversible-NoLabels; footprint promicro:ProMicro -> promicro:ProMicro-Reversible-NoLabels
- REF** (x2): value MountingHole_3.2mm_M3_Pad_Via -> MountingHole_4.6mm_Pad_Via; footprint MountingHole:MountingHole_3.2mm_M3_Pad_Via -> MountingHole:MountingHole_4.6mm_Pad_Via_Custom
- moved D35 7.94 mm to (152.4, 129.4)
- moved D34 4.76 mm to (127.0, 129.4)
- moved FACE DOWN 2.73 mm to (67.8, 57.5), turned to 0 degrees
Routing:
- net GND: track 0.00 -> 44.2 mm
- net COL2: track 165.0 -> 185.4 mm
- net COL7: track 252.3 -> 272.2 mm
- net COL5: track 218.6 -> 238.1 mm
- net COL3: track 184.3 -> 203.6 mm
- net COL4: track 174.0 -> 193.2 mm
- net VCC: track 0.00 -> 18.8 mm
- net Net-(ProMicro1-Pad24): track 0.00 -> 18.7 mm
- net Net-(ProMicro1-Pad22): track 0.00 -> 18.7 mm
- net COL6: track 208.2 -> 226.9 mm
- net COL1: track 128.0 -> 145.7 mm
- net ROW1: track 144.9 -> 159.7 mm
- net COL0: track 80.2 -> 93.6 mm
- net Net-(ProMicro1-Pad7): track 0.00 -> 12.7 mm
- net Net-(ProMicro1-Pad6): track 0.00 -> 12.7 mm
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Other:
- board text removed: "C0"
- board text removed: "C1"
- board text removed: "C2"
- board text removed: "C3"
- board text removed: "C4"
- board text removed: "C5"
- board text removed: "C6"
- board text removed: "C7"
- board text removed: "Components FACE DOWN"
- board text removed: "Components FACE UP"
- board text removed: "GND"
- board text removed: "R0"
- board text removed: "R1"
- board text removed: "R2"
- board text removed: "R3"
- board text removed: "R4"
- board text removed: "RAW"
- board text removed: "RIP AND TEAR, UNTIL IT'S DONE."
- board text removed: "RST"
- board text removed: "VCC"
