File: bottom-plate-kicad/eternal-keypad-bottom.kicad_pcb (KiCad board)
At the start: 2 copper layers, 169.9 x 95.3 mm, 7 parts

Commit message: Update plates to Kicadv6
Other:
- board size 169.9 x 95.3 mm -> 169.9 x 95.2 mm
- net class Default removed
- net class Power removed
