File: switch-plate-kicad/eternal-keypad-plate.kicad_pcb (KiCad board)
At the start: 2 copper layers, 163.5 x 95.3 mm, 44 parts

Commit message: Update plates to Kicadv6
Other:
- board size 163.5 x 95.3 mm -> 163.5 x 95.2 mm
- net class Default removed
- net class Power removed
