File: pcb-kicad/eternal-keypad.kicad_pcb (KiCad board)
At the start: 2 copper layers, 169.9 x 95.2 mm, 93 parts

Commit message: Add 3D models
Parts:
- LED1, LED2, LED3, LED4, LED5, LED6, LED7, LED8: footprint * duckyb-collection:LED_WS2812B_PLCC4_5.0x5.0mm_P3.2mm -> * duckyb-collection:LED_WS2812B_reversible
